File: PEP010-V1-Diode/PEP010-V1-Diode.kicad_pcb (KiCad board)
At the start: 2 copper layers, 45 x 45 mm, 32 parts, among them J1 Screw_Terminal_01x02, J2 Conn_01x01_Pin, J3 Conn_01x01_Pin, J4 Conn_01x01_Pin, J5 Conn_01x01_Pin, J6 Conn_01x01_Pin, J7 Conn_01x01_Pin

Commit message: Add files via upload
Parts:
- removed J3: Conn_01x01_Pin, Connector_PinHeader_2.54mm:PinHeader_1x01_P2.54mm_Vertical
- added G***: LOGO, PEP:petnica_logo, F.Cu at (127.6, 66.3)
- J1: footprint TerminalBlock_Phoenix:TerminalBlock_Phoenix_MKDS-1,5-2-5.08_1x02_P5.08mm_Horizontal -> PEP:TerminalBlock_Phoenix_MKDS-1,5-2-5.08_1x02_P5.08mm_Horizontal
- moved REF** 7.38 mm to (137.0, 100.0)
- moved REF** 4.91 mm to (123.5, 79.6)
- moved REF** 4.59 mm to (137.4, 79.1)
- moved REF** 4.42 mm to (145.0, 79.3)
- moved REF** 4.32 mm to (129.4, 79.2)
- moved J1 2.85 mm to (113.3, 80.0)
- moved REF** 1.61 mm to (137.4, 91.5)
- moved REF** 1.25 mm to (123.5, 91.6)
- moved D4 1.20 mm to (141.4, 73.0)
- moved J7 1.20 mm to (141.5, 80.0)
- moved JP4 1.20 mm to (141.5, 93.3)
- moved R4 1.20 mm to (141.5, 85.6)
- moved REF** 1.03 mm to (145.0, 91.5)
- moved R1 1.00 mm to (120.5, 85.5)
- moved D1 1.00 mm to (120.5, 73.2)
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Routing:
- net 9V: track 39.5 -> 44.5 mm
Other:
- board text added: "1K"
- board text added: "Diode"
- board text removed: "Poređenje dioda"
- board text removed: "Vin"
