File: PEP008-V1-RC_vremenska_konstanta/PEP008-V1-RC_vremenska_konstanta.kicad_pcb (KiCad board)
At the start: 2 copper layers, 45 x 45 mm, 19 parts, among them J1 Conn_01x01_Pin, J2 Screw_Terminal_01x02, J3 Conn_01x01_Pin, J4 Conn_01x01_Pin, J5 Conn_01x01_Pin, J6 Conn_01x03_Pin, J7 Conn_01x03_Pin, SW1 SW_SPDT, SW2 SW_SPDT

Commit message: Add files via upload
Parts:
- added G***: LOGO, PEP_library:petnica_logo, F.Cu at (122.5, 97.5)
- moved REF** 5.02 mm to (131.0, 97.5)
Other:
- board text added: "PEP 008"
- board text added: "Vremenska konstanta"
