File: PEP009-V1-LC_rezonantno_kolo/PEP009-V1-LC_rezonantno_kolo.kicad_pcb (KiCad board)
At the start: 2 copper layers, 45 x 45 mm, 21 parts, among them J1 Screw_Terminal_01x02, J2 Conn_01x01_Pin, J3 Conn_01x01_Pin, J4 Conn_01x01_Pin

Commit message: Add files via upload
Parts:
- removed the G*** at (137.8, 75.9)
- added G***: LOGO, PEP_library:petnica_logo, F.Cu at (143.6, 74.2)
- added G***: LOGO, PEP_library:Kalem, B.Cu at (138.8, 82.9)
